File: externals/pgbnoroute.kicad_pcb (KiCad board)
At the start: 2 copper layers, 30.7 x 49.8 mm, 13 parts, among them P1 BATT, P10 GND, P11 GND, P2 CONN_01X04, P3 CONN_01X04, P4 CONN_01X04, P5 CONN_01X04, P6 CONN_01X04, P7 CONN_01X04, P8 GND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

Commit message: final change
* remove vias to get better connectivity on GND and 5V
Routing:
- net /5V: track 110.1 -> 109.7 mm, vias 5 -> 3
Changed lines of the file:
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@@
-(kicad_pcb (version 4) (host pcbnew 4.0.4-stable)
+(kicad_pcb (version 4) (host pcbnew 4.0.6)
   (general
     (links 32)
     (no_connects 1)
-    (area 135.306999 62.408999 166.191001 112.343001)
+    (area 122.199399 57.175399 182.854602 123.164602)
     (thickness 1.6)
     (drawings 16)
-    (tracks 217)
+    (tracks 210)
     (zones 0)
     (modules 13)
@@
   (page A4)
   (layers
-    (0 F.Cu signal)
+    (0 F.Cu signal hide)
     (31 B.Cu signal)
     (33 F.Adhes user)
@@
   (segment (start 136.496 91.7414) (end 136.496 83.82) (width 1.016) (layer B.Cu) (net 3))
   (segment (start 136.496 67.4793) (end 136.496 83.82) (width 1.016) (layer B.Cu) (net 3))
-  (segment (start 138.43 74.676) (end 141.986 74.676) (width 2.54) (layer F.Cu) (net 4))
-  (segment (start 155.7338 75.946) (end 156.718 76.9302) (width 2.54) (layer F.Cu) (net 4))
-  (segment (start 153.543 75.946) (end 155.7338 75.946) (width 2.54) (layer F.Cu) (net 4))
-  (segment (start 153.416 75.819) (end 153.543 75.946) (width 2.54) (layer F.Cu) (net 4))
-  (segment (start 148.59 75.819) (end 153.416 75.819) (width 2.54) (layer F.Cu) (net 4))
-  (segment (start 148.082 76.327) (end 148.59 75.819) (width 2.54) (layer F.Cu) (net 4))
-  (via (at 148.082 76.327) (size 0.6858) (drill 0.3302) (layers F.Cu B.Cu) (net 4))
-  (segment (start 143.637 76.327) (end 148.082 76.327) (width 2.54) (layer B.Cu) (net 4))
-  (via (at 143.637 76.327) (size 0.6858) (drill 0.3302) (layers F.Cu B.Cu) (net 4))
-  (segment (start 141.986 74.676) (end 143.637 76.327) (width 2.54) (layer F.Cu) (net 4))
+  (segment (start 156.718 76.9302) (end 156.718 76.918) (width 2.54) (layer F.Cu) (net 4))
+  (segment (start 154.476 74.676) (end 138.43 74.676) (width 2.54) (layer F.Cu) (net 4))
+  (segment (start 156.718 76.918) (end 154.476 74.676) (width 2.54) (layer F.Cu) (net 4))
   (segment (start 156.718 76.9302) (end 156.718 78.994) (width 2.54) (layer F.Cu) (net 4))
   (segment (start 156.718 76.9302) (end 155.8608 76.073) (width 2.54) (layer F.Cu) (net 4))
@@
   (segment (start 157.226 77.4378) (end 157.226 78.3362) (width 2.54) (layer F.Cu) (net 4))
   (segment (start 138.43 79.756) (end 138.43 74.676) (width 2.54) (layer B.Cu) (net 4))
+  (segment (start 141.732 83.058) (end 138.43 79.756) (width 2.54) (layer B.Cu) (net 4))
+  (via (at 141.732 83.058) (size 0.6858) (drill 0.3302) (layers F.Cu B.Cu) (net 4))
+  (segment (start 141.732 90.424) (end 141.732 83.058) (width 2.54) (layer F.Cu) (net 4))
   (segment (start 140.716 91.44) (end 141.732 90.424) (width 2.54) (layer F.Cu) (net 4))
-  (segment (start 141.732 90.424) (end 141.732 83.058) (width 2.54) (layer F.Cu) (net 4))
-  (via (at 141.732 83.058) (size 0.6858) (drill 0.3302) (layers F.Cu B.Cu) (net 4))
-  (segment (start 141.732 83.058) (end 138.43 79.756) (width 2.54) (layer B.Cu) (net 4))
   (segment (start 138.43 91.44) (end 140.703 91.44) (width 2.54) (layer F.Cu) (net 4))
   (segment (start 140.957 91.694) (end 140.703 91.44) (width 2.54) (layer F.Cu) (net 4))
