File: PGP.sch (KiCad schematic (older format))
At the start: 13 parts, among them P1 BATT, P10 GND, P11 GND, P2 CONN_01X04, P3 CONN_01X04, P4 CONN_01X04, P5 CONN_01X04, P6 CONN_01X04, P7 CONN_01X04, P8 GND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

Commit message: Add files via upload
Parts:
- removed P10, P11, P8, P9: GND, Pin_Headers:Pin_Header_Straight_1x01_Pitch2.54mm, symbol CONN_01X01
Changed lines of the file:
@@
 LIBS:valves
 LIBS:5V_VOLTAGE_REGULATOR
+LIBS:PGP-cache
 EELAYER 25 0
 EELAYER END
@@
 Wire Wire Line
 	4200 1950 4200 2900
-$Comp
-L CONN_01X01 P8
-U 1 1 58E50109
-P 3600 3950
-F 0 "P8" H 3600 4050 50  0000 C CNN
-F 1 "GND" V 3700 3950 50  0000 C CNN
-F 2 "Pin_Headers:Pin_Header_Straight_1x01_Pitch2.54mm" H 3600 3950 50  0001 C CNN
-F 3 "" H 3600 3950 50  0000 C CNN
-	1    3600 3950
-	1    0    0    -1
-$EndComp
-$Comp
-L CONN_01X01 P9
-U 1 1 58E50258
-P 4050 3950
-F 0 "P9" H 4050 4050 50  0000 C CNN
-F 1 "GND" V 4150 3950 50  0000 C CNN
-F 2 "Pin_Headers:Pin_Header_Straight_1x01_Pitch2.54mm" H 4050 3950 50  0001 C CNN
-F 3 "" H 4050 3950 50  0000 C CNN
-	1    4050 3950
-	1    0    0    -1
-$EndComp
-$Comp
-L CONN_01X01 P10
-U 1 1 58E5028F
-P 4550 4000
-F 0 "P10" H 4550 4100 50  0000 C CNN
-F 1 "GND" V 4650 4000 50  0000 C CNN
-F 2 "Pin_Headers:Pin_Header_Straight_1x01_Pitch2.54mm" H 4550 4000 50  0001 C CNN
-F 3 "" H 4550 4000 50  0000 C CNN
-	1    4550 4000
-	1    0    0    -1
-$EndComp
-$Comp
-L CONN_01X01 P11
-U 1 1 58E502C7
-P 4950 4000
-F 0 "P11" H 4950 4100 50  0000 C CNN
-F 1 "GND" V 5050 4000 50  0000 C CNN
-F 2 "Pin_Headers:Pin_Header_Straight_1x01_Pitch2.54mm" H 4950 4000 50  0001 C CNN
-F 3 "" H 4950 4000 50  0000 C CNN
-	1    4950 4000
-	1    0    0    -1
-$EndComp
-$Comp
-L GND #PWR010
-U 1 1 58E503E8
-P 3400 3950
-F 0 "#PWR010" H 3400 3700 50  0001 C CNN
-F 1 "GND" H 3400 3800 50  0000 C CNN
-F 2 "" H 3400 3950 50  0000 C CNN
-F 3 "" H 3400 3950 50  0000 C CNN
-	1    3400 3950
-	0    1    1    0
-$EndComp
-$Comp
-L GND #PWR011
-U 1 1 58E50482
-P 3850 3950
-F 0 "#PWR011" H 3850 3700 50  0001 C CNN
-F 1 "GND" H 3850 3800 50  0000 C CNN
-F 2 "" H 3850 3950 50  0000 C CNN
-F 3 "" H 3850 3950 50  0000 C CNN
-	1    3850 3950
-	0    1    1    0
-$EndComp
-$Comp
-L GND #PWR012
-U 1 1 58E504B4
-P 4350 4000
-F 0 "#PWR012" H 4350 3750 50  0001 C CNN
-F 1 "GND" H 4350 3850 50  0000 C CNN
-F 2 "" H 4350 4000 50  0000 C CNN
-F 3 "" H 4350 4000 50  0000 C CNN
-	1    4350 4000
-	0    1    1    0
-$EndComp
-$Comp
-L GND #PWR013
-U 1 1 58E504E6
-P 4750 4000
-F 0 "#PWR013" H 4750 3750 50  0001 C CNN
-F 1 "GND" H 4750 3850 50  0000 C CNN
-F 2 "" H 4750 4000 50  0000 C CNN
-F 3 "" H 4750 4000 50  0000 C CNN
-	1    4750 4000
-	0    1    1    0
-$EndComp
 $EndSCHEMATC
